File: pcb/carry/Carry.kicad_pcb (KiCad board)
At the start: 2 copper layers, 21 x 28.1 mm, 9 parts, among them J2 Conn_01x02, U1 Luckfox-Pico_Mini_B, U2 MCP73831-2-OT

Commit message: updated
Routing:
- added copper zone on B.Cu, net GND
- removed copper zone on B.Cu, net (none)
- removed copper zone on F.Cu, net (none)
Other:
- board size 21 x 28.1 mm -> 21.5 x 28.6 mm
Changed lines of the file:
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@@
 		(tags "connector JST PH vertical")
 		(property "Reference" "J2"
-			(at 1 2.9 0)
+			(at -0.964259 5.39654 0)
 			(layer "B.SilkS")
 			(effects
@@
 	)
 	(gr_rect
-		(start 129 77.13)
-		(end 150 105.27)
+		(start 128.75 76.88)
+		(end 150.25 105.52)
 		(stroke
-			(width 0.05)
+			(width 0.1)
 			(type solid)
 		)
 		(fill no)
 		(layer "Edge.Cuts")
-	)
-	(segment
-		(start 138.431365 89.31434)
-		(end 138.431365 86.835965)
-		(width 0.2)
-		(layer "B.Cu")
-		(net "Net-(D1-A1)")
-	)
-	(segment
-		(start 138.431365 86.835965)
-		(end 138.567519 86.699811)
-		(width 0.2)
-		(layer "B.Cu")
-		(net "Net-(D1-A1)")
-	)
-	(segment
-		(start 139.521711 86.754003)
-		(end 139.467519 86.699811)
-		(width 0.2)
-		(layer "B.Cu")
-		(net "Net-(D1-A2)")
-	)
-	(segment
-		(start 142.187935 86.813814)
-		(end 142.128124 86.754003)
-		(width 0.2)
-		(layer "B.Cu")
-		(net "Net-(D1-A2)")
-	)
-	(segment
-		(start 142.128124 86.754003)
-		(end 139.521711 86.754003)
-		(width 0.2)
-		(layer "B.Cu")
-		(net "Net-(D1-A2)")
-	)
-	(segment
-		(start 138.431365 90.96434)
-		(end 143.001773 90.96434)
-		(width 0.2)
-		(layer "B.Cu")
-		(net "Net-(U2-STAT)")
-	)
-	(segment
-		(start 144.233492 89.732621)
-		(end 144.233492 94.405593)
-		(width 0.2)
-		(layer "B.Cu")
-		(net "Net-(U2-STAT)")
-	)
-	(segment
-		(start 144.233492 94.405593)
-		(end 144.089083 94.550002)
-		(width 0.2)
-		(layer "B.Cu")
-		(net "Net-(U2-STAT)")
-	)
-	(segment
-		(start 143.001773 90.96434)
-		(end 144.233492 89.732621)
-		(width 0.2)
-		(layer "B.Cu")
-		(net "Net-(U2-STAT)")
 	)
 	(segment
@@
 	)
 	(segment
+		(start 138.431365 89.31434)
+		(end 138.431365 86.835965)
+		(width 0.2)
+		(layer "B.Cu")
+		(net "Net-(D1-A1)")
+	)
+	(segment
+		(start 138.431365 86.835965)
+		(end 138.567519 86.699811)
+		(width 0.2)
+		(layer "B.Cu")
+		(net "Net-(D1-A1)")
+	)
+	(segment
+		(start 139.521711 86.754003)
+		(end 139.467519 86.699811)
+		(width 0.2)
+		(layer "B.Cu")
+		(net "Net-(D1-A2)")
+	)
+	(segment
+		(start 142.187935 86.813814)
+		(end 142.128124 86.754003)
+		(width 0.2)
+		(layer "B.Cu")
+		(net "Net-(D1-A2)")
+	)
+	(segment
+		(start 142.128124 86.754003)
+		(end 139.521711 86.754003)
+		(width 0.2)
+		(layer "B.Cu")
+		(net "Net-(D1-A2)")
+	)
+	(segment
+		(start 138.431365 90.96434)
+		(end 143.001773 90.96434)
+		(width 0.2)
+		(layer "B.Cu")
+		(net "Net-(U2-STAT)")
+	)
+	(segment
+		(start 144.233492 89.732621)
+		(end 144.233492 94.405593)
+		(width 0.2)
+		(layer "B.Cu")
+		(net "Net-(U2-STAT)")
+	)
+	(segment
+		(start 144.233492 94.405593)
+		(end 144.089083 94.550002)
+		(width 0.2)
+		(layer "B.Cu")
+		(net "Net-(U2-STAT)")
+	)
+	(segment
+		(start 143.001773 90.96434)
+		(end 144.233492 89.732621)
+		(width 0.2)
+		(layer "B.Cu")
+		(net "Net-(U2-STAT)")
+	)
+	(segment
 		(start 141.814083 94.550002)
 		(end 140.520936 94.550002)
@@
 	)
 	(zone
-		(layers "F.Cu" "B.Cu")
+		(net "GND")
+		(layer "B.Cu")
 		(hatch edge 0.5)
 		(connect_pads yes
-			(clearance 0.5)
+			(clearance 0.3)
 		)
 		(min_thickness 0.25)
@@
 			(thermal_gap 0.5)
 			(thermal_bridge_width 0.5)
-			(island_removal_mode 1)
+			(island_removal_mode 0)
 		)
 		(polygon
