File: pcb/carry/Carry.kicad_pcb (KiCad board)
At the start: 2 copper layers, 21.5 x 28.6 mm, 5 parts, among them U1 Luckfox-Pico_Mini_B

Commit message: finished all PCB awaiting checkup
Parts:
- added 5V1: from regulator, TestPoint:TestPoint_THTPad_D1.0mm_Drill0.5mm, F.Cu at (136.5, 79.2)
- added TP1: pin 1 of button, TestPoint:TestPoint_THTPad_D1.0mm_Drill0.5mm, F.Cu at (139.6, 79.2)
- added TP2: pin 2 of button, TestPoint:TestPoint_THTPad_D1.0mm_Drill0.5mm, F.Cu at (142.6, 79.2)
Connections:
- U1 pad 19: unconnected-(U1-GPIO4_C0_z-Pad19) -> Net-(U1-GPIO4_C0_z)
Routing:
- net Net-(U1-GPIO4_C0_z): track 0.00 -> 11.6 mm
- net Net-(U1-VBUS): track 0.14 -> 6.39 mm
- net Net-(D1-A1): track 11.3 -> 17.4 mm
- net Net-(U1-GPIO1_D3_d): track 25.5 -> 23.8 mm
