File: pcb/carry/Carry.kicad_sch (KiCad schematic)
At the start: 13 parts, among them J1 Conn_01x04_Pin, J2 Conn_01x02, U1 Luckfox-Pico_Mini_B, U2 MCP73831-2-OT

Commit message: updated
Parts:
- D1: value LED_Dual_AAK -> LED_Dual_KKA
Changed lines of the file:
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@@
+	)
+	(junction
+		(at 139.7 40.64)
+		(diameter 0)
+		(color 0 0 0 0)
 	)
 	(junction
@@
 	(wire
 		(pts
-			(xy 127 40.64) (xy 146.05 40.64)
+			(xy 127 40.64) (xy 139.7 40.64)
 		)
 		(stroke
@@
 		(pts
 			(xy 100.33 99.06) (xy 100.33 88.9)
+		)
+		(stroke
+			(width 0)
+			(type default)
+		)
+	)
+	(wire
+		(pts
+			(xy 139.7 40.64) (xy 146.05 40.64)
 		)
 		(stroke
@@
 			)
 		)
-		(property "Value" "LED_Dual_AAK"
+		(property "Value" "LED_Dual_KKA"
 			(at 200.5965 73.66 0)
 			(show_name no)
@@
 					(unit 1)
 				)
+			)
+		)
+	)
+	(symbol
+		(lib_id "power:PWR_FLAG")
+		(at 139.7 40.64 180)
+		(unit 1)
+		(body_style 1)
+		(exclude_from_sim no)
+		(in_bom yes)
+		(on_board yes)
+		(in_pos_files yes)
+		(dnp no)
+		(fields_autoplaced yes)
+		(property "Reference" "#FLG02"
+			(at 139.7 42.545 0)
+			(hide yes)
+			(show_name no)
+			(do_not_autoplace no)
+			(effects
+				(font
+					(size 1.27 1.27)
+				)
+			)
+		)
+		(property "Value" "PWR_FLAG"
+			(at 139.7 45.72 0)
+			(show_name no)
+			(do_not_autoplace no)
+			(effects
+				(font
+					(size 1.27 1.27)
+				)
+			)
+		)
+		(property "Footprint" ""
+			(at 139.7 40.64 0)
+			(hide yes)
+			(show_name no)
+			(do_not_autoplace no)
+			(effects
+				(font
+					(size 1.27 1.27)
+				)
+			)
+		)
+		(property "Datasheet" ""
+			(at 139.7 40.64 0)
+			(hide yes)
+			(show_name no)
+			(do_not_autoplace no)
+			(effects
+				(font
+					(size 1.27 1.27)
+				)
+			)
+		)
+		(property "Description" "Special symbol for telling ERC where power comes from"
+			(at 139.7 40.64 0)
+			(hide yes)
+			(show_name no)
+			(do_not_autoplace no)
+			(effects
+				(font
+					(size 1.27 1.27)
+				)
+			)
+		)
+		(pin "1"
+		)
+		(instances
+			(project "Carry"
+				(path "/460b64f1-754e-43cc-bbda-1ad83299f772"
+					(reference "#FLG02")
+					(unit 1)
+				)

Commit message: charger has been finished final draft
Parts:
- removed C1, C2: 4.7, symbol Device:C
- removed D2: D_Schottky, Diode_THT:D_DO-35_SOD27_P7.62mm_Horizontal, symbol Device:D_Schottky
- removed J1: Conn_01x04_Pin, symbol Connector:Conn_01x04_Pin
- removed J2: Conn_01x02, Connector_JST:JST_PH_B2B-PH-K_1x02_P2.00mm_Vertical, symbol Connector_Generic:Conn_01x02
- removed R1: 2k, Resistor_SMD:R_0603_1608Metric, symbol Device:R
- removed R2: 470, Resistor_SMD:R_0603_1608Metric, symbol Device:R
- removed U2: MCP73831-2-OT, Package_TO_SOT_SMD:SOT-23-5, symbol Battery_Management:MCP73831-2-OT
- added 5V1: from regulator, symbol Connector:TestPoint
- added TP1: pin 1 of button, symbol Connector:TestPoint
- added TP2: pin 2 of button, symbol Connector:TestPoint
- renumbered R3 to R1, R4 to R2
Connections:
- net GND: now also TP2.1
- net at U1.1 (VBUS): now also 5V1.1
- net at U1.19 (GPIO4_C0_z): now also TP1.1
- no-connect marks 13 -> 12
Other:
- note removed: "Battery Negative"
- note removed: "Battery Positive"
