File: pcb/dirt2/dirt.kicad_sch (KiCad schematic)
At the start: 3 parts, among them P1 USB_C_Plug_USB2.0

Commit message: uh
asdfasdfasdf
Parts:
- removed J1: (no value), symbol 4PinPogoFemale:4PinPogoFemale
- added 5V, D+, D-, GROUND, T_DIN, T_DO: TestPoint, symbol Connector:TestPoint
Connections:
- net at U1. (3v3): now also D+.1
- net at P1.A1 (GND), P1.A12 (GND), P1.B1 (GND)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: now also GROUND.1
- net at P1.A4 (VBUS), P1.A9 (VBUS), P1.B4 (VBUS)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: now also 5V.1
- new net: D-.1, U1. (3v3)
- new net: T_DIN.1, U1. (3v3)
- new net: T_DO.1, U1. (3v3)
- no-connect marks 25 -> 22
Other:
- moved on the sheet: U1
