File: pcb/dirt2/dirt.kicad_pcb (KiCad board)
At the start: 2 copper layers, 60.7 x 53.1 mm, 23 parts

Commit message: dirt finished
Other:
- outline, holes or cut-outs redrawn
Changed lines of the file:
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@@
 		(tags "test point THT pad")
 		(property "Reference" "5V_C1"
-			(at -3.85 0.102 0)
+			(at -0.02 2.322 0)
 			(layer "F.SilkS")
 			(effects
@@
 		)
 		(fp_text user "${REFERENCE}"
-			(at -3.85 0.1 0)
+			(at -0.02 2.32 0)
 			(layer "F.Fab")
 			(effects
@@
 		(tags "test point THT pad")
 		(property "Reference" "5V1"
-			(at -2.75 0.052 0)
+			(at -0.07 1.87 0)
 			(layer "F.SilkS")
 			(effects
@@
 		)
 		(fp_text user "${REFERENCE}"
-			(at -2.75 0.05 0)
+			(at -0.07 1.868 0)
 			(layer "F.Fab")
 			(effects
@@
 	)
 	(gr_line
-		(start 117.419486 82.13)
-		(end 117.419486 135.230093)
+		(start 117.441367 82.624042)
+		(end 117.404042 134.670832)
 		(stroke
 			(width 0.05)
@@
 		(layer "Edge.Cuts")
 	)
-	(gr_line
-		(start 117.419486 135.230093)
-		(end 178.12 135.23)
+	(gr_arc
+		(start 117.441367 82.624042)
+		(mid 117.6 82.25)
+		(end 117.979168 82.104042)
 		(stroke
 			(width 0.05)
@@
 		(layer "Edge.Cuts")
 	)
+	(gr_arc
+		(start 117.924042 135.208633)
+		(mid 117.55 135.05)
+		(end 117.404042 134.670832)
+		(stroke
+			(width 0.05)
+			(type default)
+		)
+		(layer "Edge.Cuts")
+	)
 	(gr_line
-		(start 178.12 82.13)
-		(end 117.419486 82.13)
+		(start 117.924042 135.208633)
+		(end 177.570832 135.245958)
+		(stroke
+			(width 0.05)
+			(type default)
+		)
+		(layer "Edge.Cuts")
+	)
+	(gr_line
+		(start 177.6 82.141367)
+		(end 117.979168 82.104042)
 		(stroke
 			(width 0.05)
@@
 		(layer "Edge.Cuts")
 	)
-	(gr_line
-		(start 178.12 135.23)
-		(end 178.12 82.13)
+	(gr_arc
+		(start 177.6 82.141367)
+		(mid 177.974042 82.3)
+		(end 178.12 82.679168)
 		(stroke
 			(width 0.05)
@@
 		(layer "Edge.Cuts")
 	)
+	(gr_arc
+		(start 178.108633 134.725958)
+		(mid 177.95 135.1)
+		(end 177.570832 135.245958)
+		(stroke
+			(width 0.05)
+			(type default)
+		)
+		(layer "Edge.Cuts")
+	)
+	(gr_line
+		(start 178.108633 134.725958)
+		(end 178.12 82.679168)
+		(stroke
+			(width 0.05)
+			(type default)
+		)
+		(layer "Edge.Cuts")
+	)
 	(segment
 		(start 132.07 107.83)
@@
 	)
 	(segment
+		(start 131.97 122.98)
+		(end 132.02 123.03)
+		(width 0.2)
+		(layer "F.Cu")
+		(net "GND")
+	)
+	(segment
+		(start 137.64 123.07)
+		(end 132.06 123.07)
+		(width 0.2)
+		(layer "F.Cu")
+		(net "GND")
+	)
+	(segment
+		(start 122.92 122.98)
+		(end 131.97 122.98)
+		(width 0.2)
+		(layer "F.Cu")
+		(net "GND")
+	)
+	(segment
+		(start 160.5 105.29)
+		(end 164.73 105.29)
+		(width 0.2)
+		(layer "F.Cu")
+		(net "GND")
+	)
+	(segment
+		(start 132.06 123.07)
+		(end 132.02 123.03)
+		(width 0.2)
+		(layer "F.Cu")
+		(net "GND")
+	)
+	(segment
+		(start 164.73 105.29)
+		(end 164.87 105.43)
+		(width 0.2)
+		(layer "F.Cu")
+		(net "GND")
+	)
+	(segment
+		(start 160.5 110.37)
+		(end 164.83 110.37)
+		(width 0.2)
+		(layer "F.Cu")
+		(net "Net-(U1-D6)")
+	)
+	(segment
+		(start 164.83 110.37)
+		(end 164.87 110.33)
+		(width 0.2)
+		(layer "F.Cu")
+		(net "Net-(U1-D6)")
+	)
+	(segment
 		(start 164.82 95.13)
 		(end 164.87 95.18)
@@
 	)
 	(segment
+		(start 132.12 102.83)
+		(end 132.32 102.83)
+		(width 0.2)
+		(layer "F.Cu")
+		(net "Net-(U1-SD1)")
+	)
+	(segment
+		(start 132.32 102.83)
+		(end 132.4 102.75)
+		(width 0.2)
+		(layer "F.Cu")
+		(net "Net-(U1-SD1)")
+	)
+	(segment
+		(start 132.4 102.75)
+		(end 137.64 102.75)
+		(width 0.2)
+		(layer "F.Cu")
+		(net "Net-(U1-SD1)")
+	)
+	(segment
+		(start 164.82 107.83)
+		(end 164.87 107.88)
+		(width 0.2)
+		(layer "F.Cu")
+		(net "Net-(U1-D5)")
+	)
+	(segment
+		(start 160.5 107.83)
+		(end 164.82 107.83)
+		(width 0.2)
+		(layer "F.Cu")
+		(net "Net-(U1-D5)")
+	)
+	(segment
+		(start 137.63 110.38)
+		(end 137.64 110.37)
+		(width 0.2)
+		(layer "F.Cu")
+		(net "Net-(U1-CLK)")
+	)
+	(segment
+		(start 132.02 110.38)
+		(end 137.63 110.38)
+		(width 0.2)
+		(layer "F.Cu")
+		(net "Net-(U1-CLK)")
+	)
+	(segment
+		(start 123.17 125.83)
+		(end 122.92 125.58)
+		(width 0.2)
+		(layer "F.Cu")
+		(net "Net-(U1-Vin)")
+	)
+	(segment
+		(start 132.02 125.83)
+		(end 123.17 125.83)
+		(width 0.2)
+		(layer "F.Cu")
+		(net "Net-(U1-Vin)")
+	)
+	(segment
+		(start 132.24 125.61)
+		(end 132.02 125.83)
+		(width 0.2)
+		(layer "F.Cu")
+		(net "Net-(U1-Vin)")
+	)
+	(segment
+		(start 137.64 125.61)
+		(end 132.24 125.61)
+		(width 0.2)
+		(layer "F.Cu")
+		(net "Net-(U1-Vin)")
+	)
+	(segment
 		(start 164.87 90.13)
 		(end 160.58 90.13)
@@
 	)
 	(segment
+		(start 164.81 97.67)
+		(end 164.87 97.73)
+		(width 0.2)
+		(layer "F.Cu")
+		(net "Net-(U1-D3)")
+	)
+	(segment
+		(start 160.5 97.67)
+		(end 164.81 97.67)
+		(width 0.2)
+		(layer "F.Cu")
+		(net "Net-(U1-D3)")
+	)
+	(segment
 		(start 160.5 100.21)
 		(end 164.79 100.21)
@@
 	)
 	(segment
-		(start 123.17 125.83)
-		(end 122.92 125.58)
-		(width 0.2)
-		(layer "F.Cu")
-		(net "Net-(U1-Vin)")
-	)
-	(segment
-		(start 132.02 125.83)
-		(end 123.17 125.83)
-		(width 0.2)
-		(layer "F.Cu")
-		(net "Net-(U1-Vin)")
-	)
-	(segment
-		(start 132.24 125.61)
-		(end 132.02 125.83)
-		(width 0.2)
-		(layer "F.Cu")
-		(net "Net-(U1-Vin)")
-	)
-	(segment
-		(start 137.64 125.61)
-		(end 132.24 125.61)
-		(width 0.2)
-		(layer "F.Cu")
-		(net "Net-(U1-Vin)")
-	)
-	(segment
-		(start 164.82 107.83)
-		(end 164.87 107.88)
-		(width 0.2)
-		(layer "F.Cu")
-		(net "Net-(U1-D5)")
-	)
-	(segment
-		(start 160.5 107.83)
-		(end 164.82 107.83)
-		(width 0.2)
-		(layer "F.Cu")
-		(net "Net-(U1-D5)")
-	)
-	(segment
-		(start 164.81 97.67)
-		(end 164.87 97.73)
-		(width 0.2)
-		(layer "F.Cu")
-		(net "Net-(U1-D3)")
-	)
-	(segment
-		(start 160.5 97.67)
-		(end 164.81 97.67)
-		(width 0.2)
-		(layer "F.Cu")
-		(net "Net-(U1-D3)")
-	)
-	(segment
 		(start 164.3 102.75)
 		(end 160.5 102.75)
@@
 		(net "Net-(U1-D8)")
 	)
-	(segment
-		(start 160.5 110.37)
-		(end 164.83 110.37)
-		(width 0.2)
-		(layer "F.Cu")
-		(net "Net-(U1-D6)")
-	)
-	(segment
-		(start 164.83 110.37)
-		(end 164.87 110.33)
-		(width 0.2)
-		(layer "F.Cu")
-		(net "Net-(U1-D6)")
-	)
-	(segment
-		(start 137.63 110.38)
-		(end 137.64 110.37)
-		(width 0.2)
-		(layer "F.Cu")
-		(net "Net-(U1-CLK)")
-	)
-	(segment
-		(start 132.02 110.38)
-		(end 137.63 110.38)
-		(width 0.2)
-		(layer "F.Cu")
-		(net "Net-(U1-CLK)")
-	)
-	(segment
-		(start 132.12 102.83)
-		(end 132.32 102.83)
-		(width 0.2)
-		(layer "F.Cu")
-		(net "Net-(U1-SD1)")
-	)
-	(segment
-		(start 132.32 102.83)
-		(end 132.4 102.75)
-		(width 0.2)
-		(layer "F.Cu")
-		(net "Net-(U1-SD1)")
-	)
-	(segment
-		(start 132.4 102.75)
-		(end 137.64 102.75)
-		(width 0.2)
-		(layer "F.Cu")
-		(net "Net-(U1-SD1)")
-	)
-	(segment
-		(start 131.97 122.98)
-		(end 132.02 123.03)
-		(width 0.2)
-		(layer "F.Cu")
-		(net "GND")
-	)
-	(segment
-		(start 137.64 123.07)
-		(end 132.06 123.07)
-		(width 0.2)
-		(layer "F.Cu")
-		(net "GND")
-	)
-	(segment
-		(start 122.92 122.98)
-		(end 131.97 122.98)
-		(width 0.2)
-		(layer "F.Cu")
-		(net "GND")
-	)
-	(segment
-		(start 160.5 105.29)
-		(end 164.73 105.29)
-		(width 0.2)
-		(layer "F.Cu")
-		(net "GND")
-	)
-	(segment
-		(start 132.06 123.07)
-		(end 132.02 123.03)
-		(width 0.2)
-		(layer "F.Cu")
-		(net "GND")
-	)
-	(segment
-		(start 164.73 105.29)
-		(end 164.87 105.43)
-		(width 0.2)
-		(layer "F.Cu")
-		(net "GND")
-	)
 	(zone
