File: pcb/dirt2/.history/dirt.kicad_sch (KiCad schematic)
At the start: 4 parts, among them P1 USB_C_Plug_USB2.0

Commit message: uh
asdfasdfasdf
Parts:
- removed J1: (no value), symbol 4PinPogoFemale:4PinPogoFemale
- removed QD3203-RY1: QD3203-RY, QD3203-RY, symbol 2.8inch_MSP2807_Schematic_Package_Library:FPC240A8230-V1-E
- added 5V, D+, D-, GROUND, T_DIN, T_DO: TestPoint, symbol Connector:TestPoint
Connections:
- net at U1. (3v3): now also D+.1
- net at P1.A4 (VBUS), P1.A9 (VBUS), P1.B4 (VBUS)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: now also 5V.1
- net GND: no longer names the net of P1.A1 (GND), P1.A12 (GND), P1.B1 (GND), P1.B12 (GND), U1. (3v3)
- net GND: now also GROUND.1
- new net: D-.1, U1. (3v3)
- new net: T_DIN.1, U1. (3v3)
- new net: T_DO.1, U1. (3v3)
- no-connect marks 23 -> 22
Other:
- moved on the sheet: U1

Commit message: i created some edits and added the zine
Parts:
- removed P1: USB_C_Plug_USB2.0, symbol Connector:USB_C_Plug_USB2.0
- added 3.3V_LCD1: 3.3V Output to LCD, TestPoint:TestPoint_THTPad_D1.0mm_Drill0.5mm, symbol Connector:TestPoint
- added 5V_C1: 5V Input USB C, TestPoint:TestPoint_THTPad_D1.0mm_Drill0.5mm, symbol Connector:TestPoint
- added D+_Pogo1: D+ FROM Pogo, TestPoint:TestPoint_THTPad_D1.0mm_Drill0.5mm, symbol Connector:TestPoint
- added D-_Pogo1: D- FROM Pogo, TestPoint:TestPoint_THTPad_D1.0mm_Drill0.5mm, symbol Connector:TestPoint
- added GROUND_C1: GND from USB C, TestPoint:TestPoint_THTPad_D1.0mm_Drill0.5mm, symbol Connector:TestPoint
- added GROUND_LCD1: GND to LCD, TestPoint:TestPoint_THTPad_D1.0mm_Drill0.5mm, symbol Connector:TestPoint
- added TBD1, TBD2, TBD3, TBD4, TBD5: TestPoint, symbol Connector:TestPoint
- added T_CLK1: TestPoint, TestPoint:TestPoint_THTPad_D1.0mm_Drill0.5mm, symbol Connector:TestPoint
- 5V1: renamed from 5V; value TestPoint -> 5V Output from Pogo; footprint (none) -> TestPoint:TestPoint_THTPad_D1.0mm_Drill0.5mm
- D+_C1: renamed from D+; value TestPoint -> D+ FROM USB C; footprint (none) -> TestPoint:TestPoint_THTPad_D1.0mm_Drill0.5mm
- D-_C1: renamed from D-; value TestPoint -> D- FROM USB C; footprint (none) -> TestPoint:TestPoint_THTPad_D1.0mm_Drill0.5mm
- GROUND1: renamed from GROUND; value TestPoint -> GND from Pogo; footprint (none) -> TestPoint:TestPoint_THTPad_D1.0mm_Drill0.5mm
- T_DIN1: renamed from T_DIN; footprint (none) -> TestPoint:TestPoint_THTPad_D1.0mm_Drill0.5mm
- T_DO1: renamed from T_DO; footprint (none) -> TestPoint:TestPoint_THTPad_D1.0mm_Drill0.5mm
Connections:
- net at GROUND1.1: now also U1.J1_14 (GND), GROUND_C1.1; no longer U1. (3v3)
- net at D-_C1.1: now also U1.J2_4 (D3); no longer U1. (3v3)
- net at T_DIN1.1: now also U1.J1_8 (SD0); no longer U1. (3v3)
- net at 5V1.1: now also U1.J1_15 (Vin), 5V_C1.1; no longer U1. (3v3)
- net at T_DO1.1: now also U1.J1_6 (SD1); no longer U1. (3v3)
- net at D+_C1.1: now also U1.J2_3 (D2); no longer U1. (3v3)
- new net: T_CLK1.1, U1.J1_9 (CLK)
- new net: D+_Pogo1.1, U1.J2_1 (D0)
- new net: TBD3.1, U1.J2_10 (D7)
- new net: TBD4.1, U1.J2_11 (D8)
- new net: D-_Pogo1.1, U1.J2_2 (D1)
- new net: TBD5.1, U1.J2_5 (D4)
- new net: 3.3V_LCD1.1, U1.J2_6 (3v3)
- new net: GROUND_LCD1.1, U1.J2_7 (GND)
- new net: TBD1.1, U1.J2_8 (D5)
- new net: TBD2.1, U1.J2_9 (D6)
- no-connect marks 22 -> 14
Other:
- moved on the sheet: 5V1, D+_C1, D-_C1, GROUND1, T_DIN1, T_DO1

Commit message: charger has been finished final draft
Parts:
- added LED1: TestPoint, symbol Connector:TestPoint
- CS1: renamed from TBD3; footprint (none) -> TestPoint:TestPoint_THTPad_D1.0mm_Drill0.5mm
- RS1: renamed from TBD4; footprint (none) -> TestPoint:TestPoint_THTPad_D1.0mm_Drill0.5mm
- SCK1: renamed from TBD2; footprint (none) -> TestPoint:TestPoint_THTPad_D1.0mm_Drill0.5mm
- SDI1: renamed from TBD1; footprint (none) -> TestPoint:TestPoint_THTPad_D1.0mm_Drill0.5mm
- SDO1: renamed from TBD5; footprint (none) -> TestPoint:TestPoint_THTPad_D1.0mm_Drill0.5mm
Connections:
- net GND: now reaches GROUND1.1, GROUND_C1.1, U1.J1_14 (GND)
- net GND: now also GROUND_LCD1.1, U1.J2_7 (GND)
- net at U1.J2_15 (3v3): now also LED1.1
- no-connect marks 14 -> 13
Other:
- moved on the sheet: GROUND_LCD1
