File: pcb/dirt2/.history/dirt.kicad_pcb (KiCad board)
At the start: 2 copper layers, 1 part

Commit message: i created some edits and added the zine
Parts:
- removed REF**: SEEED_113990105, esp8622footprint:SEEED_113990105
- added 3.3V_LCD1: 3.3V Output to LCD, TestPoint:TestPoint_THTPad_D1.0mm_Drill0.5mm, F.Cu at (174.9, 58.8)
- added 5V1: 5V Output from Pogo, TestPoint:TestPoint_THTPad_D1.0mm_Drill0.5mm, F.Cu at (133.0, 81.6)
- added 5V_C1: 5V Input USB C, TestPoint:TestPoint_THTPad_D1.0mm_Drill0.5mm, F.Cu at (142.1, 81.8)
- added D+_C1: D+ FROM USB C, TestPoint:TestPoint_THTPad_D1.0mm_Drill0.5mm, F.Cu at (174.9, 51.2)
- added D+_Pogo1: D+ FROM Pogo, TestPoint:TestPoint_THTPad_D1.0mm_Drill0.5mm, F.Cu at (174.9, 46.1)
- added D-_C1: D- FROM USB C, TestPoint:TestPoint_THTPad_D1.0mm_Drill0.5mm, F.Cu at (174.9, 53.8)
- added D-_Pogo1: D- FROM Pogo, TestPoint:TestPoint_THTPad_D1.0mm_Drill0.5mm, F.Cu at (174.9, 48.6)
- added GROUND1: GND from Pogo, TestPoint:TestPoint_THTPad_D1.0mm_Drill0.5mm, F.Cu at (142.1, 79.0)
- added GROUND_C1: GND from USB C, TestPoint:TestPoint_THTPad_D1.0mm_Drill0.5mm, F.Cu at (133.0, 79.0)
- added GROUND_LCD1: GND to LCD, TestPoint:TestPoint_THTPad_D1.0mm_Drill0.5mm, F.Cu at (174.9, 61.5)
- added T_CLK1: TestPoint, TestPoint:TestPoint_THTPad_D1.0mm_Drill0.5mm, F.Cu at (142.1, 66.4)
- added T_DIN1: TestPoint, TestPoint:TestPoint_THTPad_D1.0mm_Drill0.5mm, F.Cu at (142.2, 63.9)
- added T_DO1: TestPoint, TestPoint:TestPoint_THTPad_D1.0mm_Drill0.5mm, F.Cu at (142.2, 58.9)
- added U1: ~, esp8622footprint:SEEED_113990105, F.Cu at (159.2, 63.9)
Other:
- board outline added: 60.7 x 53.1 mm

Commit message: charger has been finished final draft
Parts:
- added ?: , , F.Cu at (174.7, 85.3)
- added ?: , , F.Cu at (174.8, 131.4)
- added ?: , , F.Cu at (120.9, 131.6)
- added ?: , , F.Cu at (121.0, 85.6)
- added CS1: TestPoint, TestPoint:TestPoint_THTPad_D1.0mm_Drill0.5mm, F.Cu at (164.9, 112.8)
- added RS1: TestPoint, TestPoint:TestPoint_THTPad_D1.0mm_Drill0.5mm, F.Cu at (164.9, 115.4)
- added SCK1: TestPoint, TestPoint:TestPoint_THTPad_D1.0mm_Drill0.5mm, F.Cu at (164.9, 110.3)
- added SDI1: TestPoint, TestPoint:TestPoint_THTPad_D1.0mm_Drill0.5mm, F.Cu at (164.9, 107.9)
- added SDO1: TestPoint, TestPoint:TestPoint_THTPad_D1.0mm_Drill0.5mm, F.Cu at (164.9, 100.1)
- moved T_DIN1 45.1 mm to (132.1, 107.8)
- moved U1 45.1 mm to (149.1, 107.8)
- moved 3.3V_LCD1 45.1 mm to (164.9, 102.7)
- moved 5V1 45.1 mm to (122.9, 125.6)
- moved 5V_C1 45.1 mm to (132.0, 125.8)
- moved D+_C1 45.1 mm to (164.9, 95.2)
- moved D-_C1 45.1 mm to (164.9, 97.7)
- moved GROUND1 45.1 mm to (132.0, 123.0)
- moved GROUND_C1 45.1 mm to (122.9, 123.0)
- moved GROUND_LCD1 45.1 mm to (164.9, 105.4)
- moved D+_Pogo1 45.1 mm to (164.9, 90.1)
- moved D-_Pogo1 45.1 mm to (164.9, 92.6)
- moved T_DO1 45.1 mm to (132.1, 102.8)
- moved T_CLK1 45.1 mm to (132.0, 110.4)
Connections:
- GROUND1 pad 1: Net-(U1-D1)_1 -> GND
- GROUND_C1 pad 1: Net-(U1-D1)_1 -> GND
- GROUND_LCD1 pad 1: Net-(U1-D5)_1 -> GND
- U1 pad J1_14: Net-(U1-D1)_1 -> GND
- U1 pad J2_15: unconnected-(U1-3v3-PadJ2_15) -> Net-(LED1-Pad1)
- U1 pad J2_7: Net-(U1-D5)_1 -> GND
Routing:
- net GND: track 0.00 -> 19.2 mm
- net Net-(U1-Vin): track 0.00 -> 14.9 mm
- net Net-(U1-CLK): track 0.00 -> 5.62 mm
- net Net-(U1-SD0): track 0.00 -> 5.57 mm
- net Net-(U1-SD1): track 0.00 -> 5.55 mm
- net Net-(U1-D4): track 0.00 -> 4.47 mm
- net Net-(U1-D7): track 0.00 -> 4.42 mm
- net Net-(U1-D0): track 0.00 -> 4.40 mm
- net Net-(U1-D3): track 0.00 -> 4.39 mm
- net Net-(U1-D2): track 0.00 -> 4.39 mm
- net Net-(U1-D5): track 0.00 -> 4.39 mm
- net Net-(U1-D6): track 0.00 -> 4.39 mm
- net Net-(3.3V_LCD1-Pad1): track 0.00 -> 4.38 mm
- net Net-(U1-D8): track 0.00 -> 4.38 mm
- net Net-(U1-D1): track 0.00 -> 4.37 mm
- added copper zone on F.Cu, net GND

Commit message: dirt finished
Other:
- outline, holes or cut-outs redrawn
Changed lines of the file:
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@@
 		(tags "test point THT pad")
 		(property "Reference" "5V_C1"
-			(at -3.85 0.102 0)
+			(at -0.02 2.322 0)
 			(layer "F.SilkS")
 			(effects
@@
 		)
 		(fp_text user "${REFERENCE}"
-			(at -3.85 0.1 0)
+			(at -0.02 2.32 0)
 			(layer "F.Fab")
 			(effects
@@
 		(tags "test point THT pad")
 		(property "Reference" "5V1"
-			(at -2.75 0.052 0)
+			(at -0.07 1.87 0)
 			(layer "F.SilkS")
 			(effects
@@
 		)
 		(fp_text user "${REFERENCE}"
-			(at -2.75 0.05 0)
+			(at -0.07 1.868 0)
 			(layer "F.Fab")
 			(effects
@@
 	)
 	(gr_line
-		(start 117.419486 82.13)
-		(end 117.419486 135.230093)
+		(start 117.441367 82.624042)
+		(end 117.404042 134.670832)
 		(stroke
 			(width 0.05)
@@
 		(layer "Edge.Cuts")
 	)
-	(gr_line
-		(start 117.419486 135.230093)
-		(end 178.12 135.23)
+	(gr_arc
+		(start 117.441367 82.624042)
+		(mid 117.6 82.25)
+		(end 117.979168 82.104042)
 		(stroke
 			(width 0.05)
@@
 		(layer "Edge.Cuts")
 	)
+	(gr_arc
+		(start 117.924042 135.208633)
+		(mid 117.55 135.05)
+		(end 117.404042 134.670832)
+		(stroke
+			(width 0.05)
+			(type default)
+		)
+		(layer "Edge.Cuts")
+	)
 	(gr_line
-		(start 178.12 82.13)
+		(start 117.924042 135.208633)
+		(end 177.570832 135.245958)
+		(stroke
+			(width 0.05)
+			(type default)
+		)
+		(layer "Edge.Cuts")
+	)
+	(gr_line
+		(start 177.6 82.141367)
 		(end 117.419486 82.13)
 		(stroke
@@
 		(layer "Edge.Cuts")
 	)
-	(gr_line
-		(start 178.12 135.23)
-		(end 178.12 82.13)
+	(gr_arc
+		(start 177.6 82.141367)
+		(mid 177.974042 82.3)
+		(end 178.12 82.679168)
 		(stroke
 			(width 0.05)
@@
 		(layer "Edge.Cuts")
 	)
+	(gr_arc
+		(start 178.108633 134.725958)
+		(mid 177.95 135.1)
+		(end 177.570832 135.245958)
+		(stroke
+			(width 0.05)
+			(type default)
+		)
+		(layer "Edge.Cuts")
+	)
+	(gr_line
+		(start 178.108633 134.725958)
+		(end 178.12 82.679168)
+		(stroke
+			(width 0.05)
+			(type default)
+		)
+		(layer "Edge.Cuts")
+	)
 	(segment
 		(start 132.07 107.83)
@@
 	)
 	(segment
+		(start 131.97 122.98)
+		(end 132.02 123.03)
+		(width 0.2)
+		(layer "F.Cu")
+		(net "GND")
+	)
+	(segment
+		(start 137.64 123.07)
+		(end 132.06 123.07)
+		(width 0.2)
+		(layer "F.Cu")
+		(net "GND")
+	)
+	(segment
+		(start 122.92 122.98)
+		(end 131.97 122.98)
+		(width 0.2)
+		(layer "F.Cu")
+		(net "GND")
+	)
+	(segment
+		(start 160.5 105.29)
+		(end 164.73 105.29)
+		(width 0.2)
+		(layer "F.Cu")
+		(net "GND")
+	)
+	(segment
+		(start 132.06 123.07)
+		(end 132.02 123.03)
+		(width 0.2)
+		(layer "F.Cu")
+		(net "GND")
+	)
+	(segment
+		(start 164.73 105.29)
+		(end 164.87 105.43)
+		(width 0.2)
+		(layer "F.Cu")
+		(net "GND")
+	)
+	(segment
+		(start 160.5 110.37)
+		(end 164.83 110.37)
+		(width 0.2)
+		(layer "F.Cu")
+		(net "Net-(U1-D6)")
+	)
+	(segment
+		(start 164.83 110.37)
+		(end 164.87 110.33)
+		(width 0.2)
+		(layer "F.Cu")
+		(net "Net-(U1-D6)")
+	)
+	(segment
 		(start 164.82 95.13)
 		(end 164.87 95.18)
@@
 	)
 	(segment
+		(start 132.12 102.83)
+		(end 132.32 102.83)
+		(width 0.2)
+		(layer "F.Cu")
+		(net "Net-(U1-SD1)")
+	)
+	(segment
+		(start 132.32 102.83)
+		(end 132.4 102.75)
+		(width 0.2)
+		(layer "F.Cu")
+		(net "Net-(U1-SD1)")
+	)
+	(segment
+		(start 132.4 102.75)
+		(end 137.64 102.75)
+		(width 0.2)
+		(layer "F.Cu")
+		(net "Net-(U1-SD1)")
+	)
+	(segment
+		(start 164.82 107.83)
+		(end 164.87 107.88)
+		(width 0.2)
+		(layer "F.Cu")
+		(net "Net-(U1-D5)")
+	)
+	(segment
+		(start 160.5 107.83)
+		(end 164.82 107.83)
+		(width 0.2)
+		(layer "F.Cu")
+		(net "Net-(U1-D5)")
+	)
+	(segment
+		(start 137.63 110.38)
+		(end 137.64 110.37)
+		(width 0.2)
+		(layer "F.Cu")
+		(net "Net-(U1-CLK)")
+	)
+	(segment
+		(start 132.02 110.38)
+		(end 137.63 110.38)
+		(width 0.2)
+		(layer "F.Cu")
+		(net "Net-(U1-CLK)")
+	)
+	(segment
+		(start 123.17 125.83)
+		(end 122.92 125.58)
+		(width 0.2)
+		(layer "F.Cu")
+		(net "Net-(U1-Vin)")
+	)
+	(segment
+		(start 132.02 125.83)
+		(end 123.17 125.83)
+		(width 0.2)
+		(layer "F.Cu")
+		(net "Net-(U1-Vin)")
+	)
+	(segment
+		(start 132.24 125.61)
+		(end 132.02 125.83)
+		(width 0.2)
+		(layer "F.Cu")
+		(net "Net-(U1-Vin)")
+	)
+	(segment
+		(start 137.64 125.61)
+		(end 132.24 125.61)
+		(width 0.2)
+		(layer "F.Cu")
+		(net "Net-(U1-Vin)")
+	)
+	(segment
 		(start 164.87 90.13)
 		(end 160.58 90.13)
@@
 	)
 	(segment
+		(start 164.81 97.67)
+		(end 164.87 97.73)
+		(width 0.2)
+		(layer "F.Cu")
+		(net "Net-(U1-D3)")
+	)
+	(segment
+		(start 160.5 97.67)
+		(end 164.81 97.67)
+		(width 0.2)
+		(layer "F.Cu")
+		(net "Net-(U1-D3)")
+	)
+	(segment
 		(start 160.5 100.21)
 		(end 164.79 100.21)
@@
 	)
 	(segment
-		(start 123.17 125.83)
-		(end 122.92 125.58)
-		(width 0.2)
-		(layer "F.Cu")
-		(net "Net-(U1-Vin)")
-	)
-	(segment
-		(start 132.02 125.83)
-		(end 123.17 125.83)
-		(width 0.2)
-		(layer "F.Cu")
-		(net "Net-(U1-Vin)")
-	)
-	(segment
-		(start 132.24 125.61)
-		(end 132.02 125.83)
-		(width 0.2)
-		(layer "F.Cu")
-		(net "Net-(U1-Vin)")
-	)
-	(segment
-		(start 137.64 125.61)
-		(end 132.24 125.61)
-		(width 0.2)
-		(layer "F.Cu")
-		(net "Net-(U1-Vin)")
-	)
-	(segment
-		(start 164.82 107.83)
-		(end 164.87 107.88)
-		(width 0.2)
-		(layer "F.Cu")
-		(net "Net-(U1-D5)")
-	)
-	(segment
-		(start 160.5 107.83)
-		(end 164.82 107.83)
-		(width 0.2)
-		(layer "F.Cu")
-		(net "Net-(U1-D5)")
-	)
-	(segment
-		(start 164.81 97.67)
-		(end 164.87 97.73)
-		(width 0.2)
-		(layer "F.Cu")
-		(net "Net-(U1-D3)")
-	)
-	(segment
-		(start 160.5 97.67)
-		(end 164.81 97.67)
-		(width 0.2)
-		(layer "F.Cu")
-		(net "Net-(U1-D3)")
-	)
-	(segment
 		(start 164.3 102.75)
 		(end 160.5 102.75)
@@
 		(net "Net-(U1-D8)")
 	)
-	(segment
-		(start 160.5 110.37)
-		(end 164.83 110.37)
-		(width 0.2)
-		(layer "F.Cu")
-		(net "Net-(U1-D6)")
-	)
-	(segment
-		(start 164.83 110.37)
-		(end 164.87 110.33)
-		(width 0.2)
-		(layer "F.Cu")
-		(net "Net-(U1-D6)")
-	)
-	(segment
-		(start 137.63 110.38)
-		(end 137.64 110.37)
-		(width 0.2)
-		(layer "F.Cu")
-		(net "Net-(U1-CLK)")
-	)
-	(segment
-		(start 132.02 110.38)
-		(end 137.63 110.38)
-		(width 0.2)
-		(layer "F.Cu")
-		(net "Net-(U1-CLK)")
-	)
-	(segment
-		(start 132.12 102.83)
-		(end 132.32 102.83)
-		(width 0.2)
-		(layer "F.Cu")
-		(net "Net-(U1-SD1)")
-	)
-	(segment
-		(start 132.32 102.83)
-		(end 132.4 102.75)
-		(width 0.2)
-		(layer "F.Cu")
-		(net "Net-(U1-SD1)")
-	)
-	(segment
-		(start 132.4 102.75)
-		(end 137.64 102.75)
-		(width 0.2)
-		(layer "F.Cu")
-		(net "Net-(U1-SD1)")
-	)
-	(segment
-		(start 131.97 122.98)
-		(end 132.02 123.03)
-		(width 0.2)
-		(layer "F.Cu")
-		(net "GND")
-	)
-	(segment
-		(start 137.64 123.07)
-		(end 132.06 123.07)
-		(width 0.2)
-		(layer "F.Cu")
-		(net "GND")
-	)
-	(segment
-		(start 122.92 122.98)
-		(end 131.97 122.98)
-		(width 0.2)
-		(layer "F.Cu")
-		(net "GND")
-	)
-	(segment
-		(start 160.5 105.29)
-		(end 164.73 105.29)
-		(width 0.2)
-		(layer "F.Cu")
-		(net "GND")
-	)
-	(segment
-		(start 132.06 123.07)
-		(end 132.02 123.03)
-		(width 0.2)
-		(layer "F.Cu")
-		(net "GND")
-	)
-	(segment
-		(start 164.73 105.29)
-		(end 164.87 105.43)
-		(width 0.2)
-		(layer "F.Cu")
-		(net "GND")
-	)
 	(zone
