File: pcb/carry/.history/Carry.kicad_pcb (KiCad board)
At the start: 2 copper layers, 22.9 x 30.5 mm, 9 parts, among them J2 Conn_01x02, U1 Luckfox-Pico_Mini_B, U2 MCP73831-2-OT

Commit message: updated
Parts:
- D1, J2, MK1, R1, R2, R3, R4, U2: moved to B.Cu
- moved R2 39.3 mm to (145.1, 89.7), turned to 0 degrees
- moved J2 36.1 mm to (142.5, 80.0), turned to 180 degrees
- moved MK1 35.3 mm to (139.1, 101.0), turned to 180 degrees
- moved U2 33.3 mm to (143.0, 95.5), turned to 180 degrees
- moved R3 30.9 mm to (143.0, 86.8), turned to 0 degrees
- moved U1 30.0 mm to (139.5, 91.2)
- moved R4 29.3 mm to (138.4, 90.1), turned to 90 degrees
- moved D1 25.4 mm to (139.0, 86.2), turned to 180 degrees
- moved R1 25.2 mm to (139.0, 93.8), turned to 0 degrees
Routing:
- net Net-(J1-Pin_1): track 31.0 -> 40.5 mm, vias 0 -> 1
- net Net-(MK1-WS): track 3.92 -> 11.4 mm, vias 0 -> 1
- net /MIC_DATA: track 6.02 -> 13.3 mm, vias 0 -> 2
- net Net-(MK1-VDD): track 14.1 -> 19.8 mm
- net Net-(U2-STAT): track 6.70 -> 11.2 mm
- net Net-(D1-A2): track 6.45 -> 2.77 mm
- net Net-(MK1-BCLK): track 13.5 -> 10.4 mm
- net Net-(D1-A1): track 4.55 -> 2.67 mm
- added copper zone on B.Cu, net GND
- removed copper zone on F.Cu, net Net-(MK1-BCLK)
Other:
- board size 22.9 x 30.5 mm -> 21.5 x 28.6 mm

Commit message: charger has been finished final draft
Parts:
- removed J2: Conn_01x02, Connector_JST:JST_PH_B2B-PH-K_1x02_P2.00mm_Vertical
- removed R3: 330, Resistor_SMD:R_0603_1608Metric
- removed R4: 1k, Resistor_SMD:R_0603_1608Metric
- removed U2: MCP73831-2-OT, Package_TO_SOT_SMD:SOT-23-5
- D1: value LED_Dual_AAK -> LED_Dual_KKA
- R1: value 2k -> 1k
- R2: value 470 -> 1k
Connections:
- R1 pad 1: GND -> Net-(U1-GPIO1_D3_d)
- R1 pad 2: Net-(U2-PROG) -> Net-(D1-A2)
- R2 pad 1: Net-(U2-STAT) -> Net-(D1-A1)
- R2 pad 2: Net-(J1-Pin_1) -> Net-(U1-GPIO1_D2_d)
- U1 pad 1: Net-(J1-Pin_1) -> Net-(U1-VBUS)
- U1 pad 14: unconnected-(U1-GPIO1_D2_d-Pad14) -> Net-(U1-GPIO1_D2_d)
- U1 pad 15: unconnected-(U1-GPIO1_D3_d-Pad15) -> Net-(U1-GPIO1_D3_d)
- U1 pad 20: Net-(U1-GPIO4_C1_z) -> unconnected-(U1-GPIO4_C1_z-Pad20)
Routing:
- net Net-(J1-Pin_1): track 40.5 -> 0.00 mm, vias 1 -> 0
- net Net-(U1-GPIO1_D3_d): track 0.00 -> 25.5 mm
- net Net-(U2-STAT): track 11.2 -> 0.00 mm
- net Net-(U1-GPIO1_D2_d): track 0.00 -> 10.1 mm
- net Net-(D1-A1): track 2.67 -> 11.3 mm
- net Net-(U1-GPIO4_C1_z): track 5.86 -> 0.00 mm
- net Net-(D1-A2): track 2.77 -> 7.29 mm
- net Net-(U2-PROG): track 2.29 -> 0.00 mm

Commit message: finished all PCB awaiting checkup
Parts:
- added 5V1: from regulator, TestPoint:TestPoint_THTPad_D1.0mm_Drill0.5mm, F.Cu at (136.5, 79.2)
- added TP1: pin 1 of button, TestPoint:TestPoint_THTPad_D1.0mm_Drill0.5mm, F.Cu at (139.6, 79.2)
- added TP2: pin 2 of button, TestPoint:TestPoint_THTPad_D1.0mm_Drill0.5mm, F.Cu at (142.6, 79.2)
Connections:
- U1 pad 19: unconnected-(U1-GPIO4_C0_z-Pad19) -> Net-(U1-GPIO4_C0_z)
Routing:
- net Net-(U1-GPIO4_C0_z): track 0.00 -> 11.6 mm
- net Net-(U1-VBUS): track 0.14 -> 6.39 mm
- net Net-(D1-A1): track 11.3 -> 17.4 mm
- net Net-(U1-GPIO1_D3_d): track 25.5 -> 23.8 mm
