File: pcb/carry/.history/Carry.kicad_sch (KiCad schematic)
At the start: 12 parts, among them J1 Conn_01x04_Pin, J2 Conn_01x02, U1 Luckfox-Pico_Mini_B, U2 MCP73831-2-OT

Commit message: updated
Parts:
- added D2: D_Schottky, Diode_THT:D_DO-35_SOD27_P7.62mm_Horizontal, symbol Device:D_Schottky
- R3: value 330 -> 1k; footprint Resistor_SMD:R_0603_1608Metric -> (none)
- R4: footprint Resistor_SMD:R_0603_1608Metric -> (none)
Connections:
- net at C1.1, J1.1 (Pin_1), R2.2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: now also D2.1 (K); no longer C2.1, J2.1 (Pin_1), U2.3 (V_{BAT})
- net at D1.1 (A1): now also R4.1; no longer R4.2
- net at D1.2 (A2): now also R3.2; no longer R3.1
- net at U1.14 (GPIO1_D2_d): now also R4.2
- net at U1.15 (GPIO1_D3_d): now also R3.1
- net at U1.20 (GPIO4_C1_z): no longer R3.2
- net at R2.1, U2.1 (STAT): no longer R4.1
- net D+: no longer names the net of J1.3 (Pin_3)
- net D-: no longer names the net of J1.2 (Pin_2)
- new net: C2.1, D2.2 (A), J2.1 (Pin_1), U2.3 (V_{BAT})
- no-connect marks 16 -> 13
Other:
- moved on the sheet: D1

Commit message: updated
Parts:
- D1: value LED_Dual_AAK -> LED_Dual_KKA
Changed lines of the file:
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@@
 			)
 		)
-		(property "Value" "LED_Dual_AAK"
+		(property "Value" "LED_Dual_KKA"
 			(at 200.5965 73.66 0)
 			(show_name no)

Commit message: charger has been finished final draft
Parts:
- removed C1, C2: 4.7, symbol Device:C
- removed D2: D_Schottky, Diode_THT:D_DO-35_SOD27_P7.62mm_Horizontal, symbol Device:D_Schottky
- removed J1: Conn_01x04_Pin, symbol Connector:Conn_01x04_Pin
- removed J2: Conn_01x02, Connector_JST:JST_PH_B2B-PH-K_1x02_P2.00mm_Vertical, symbol Connector_Generic:Conn_01x02
- removed R1: 2k, Resistor_SMD:R_0603_1608Metric, symbol Device:R
- removed R2: 470, Resistor_SMD:R_0603_1608Metric, symbol Device:R
- removed U2: MCP73831-2-OT, Package_TO_SOT_SMD:SOT-23-5, symbol Battery_Management:MCP73831-2-OT
- added 5V1: from regulator, symbol Connector:TestPoint
- added TP1: pin 1 of button, symbol Connector:TestPoint
- added TP2: pin 2 of button, symbol Connector:TestPoint
- renumbered R3 to R1, R4 to R2
Connections:
- net GND: now also TP2.1
- net at U1.1 (VBUS): now also 5V1.1
- net at U1.19 (GPIO4_C0_z): now also TP1.1
- no-connect marks 13 -> 12
Other:
- note removed: "Battery Negative"
- note removed: "Battery Positive"

Commit message: finished all PCB awaiting checkup
Parts:
- 5V1, TP1, TP2: footprint (none) -> TestPoint:TestPoint_THTPad_D1.0mm_Drill0.5mm
Changed lines of the file:
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@@
 			)
 		)
-		(property "Footprint" ""
+		(property "Footprint" "TestPoint:TestPoint_THTPad_D1.0mm_Drill0.5mm"
 			(at 134.62 55.88 0)
 			(hide yes)
@@
 			)
 		)
-		(property "Footprint" ""
+		(property "Footprint" "TestPoint:TestPoint_THTPad_D1.0mm_Drill0.5mm"
 			(at 189.23 73.66 0)
 			(hide yes)
@@
 			)
 		)
-		(property "Footprint" ""
+		(property "Footprint" "TestPoint:TestPoint_THTPad_D1.0mm_Drill0.5mm"
 			(at 209.55 63.5 0)
 			(hide yes)
